File: A600-DB9-Relocator.kicad_pcb (KiCad board)
At the start: 2 copper layers, 3 parts, among them J1 DB9_Female, J2 DB9_Female, J3 DB9-Dual-Male

Commit message: PCB complete
Parts:
- added J4: Conn_02x09_Odd_Even, Connector_PinHeader_2.54mm:PinHeader_2x09_P2.54mm_Vertical, F.Cu at (122.0, 30.0)
- added J5: Conn_02x09_Odd_Even, Connector_PinHeader_2.54mm:PinHeader_2x09_P2.54mm_Vertical, F.Cu at (122.0, 93.0)
- added MECH: PinSocket_2x02_P2.54mm_Vertical, Connector_PinSocket_2.54mm:PinSocket_2x02_P2.54mm_Vertical, F.Cu at (122.0, 143.0)
- added MECH: PinSocket_2x02_P2.54mm_Vertical, Connector_PinSocket_2.54mm:PinSocket_2x02_P2.54mm_Vertical, F.Cu at (122.0, 80.0)
- moved J3 141.1 mm to (120.7, 269.2)
- moved J2 6.96 mm to (130.0, 35.0)
- moved J1 6.86 mm to (130.0, 66.5)
Connections:
- J3 pad A1: Net-(J1-Pad1) -> Net-(J3-PadA1)
- J3 pad A2: Net-(J1-Pad2) -> Net-(J3-PadA2)
- J3 pad A3: Net-(J1-Pad3) -> Net-(J3-PadA3)
- J3 pad A4: Net-(J1-Pad4) -> Net-(J3-PadA4)
- J3 pad A5: Net-(J1-Pad5) -> Net-(J3-PadA5)
- J3 pad A6: Net-(J1-Pad6) -> Net-(J3-PadA6)
- J3 pad A7: Net-(J1-Pad7) -> Net-(J3-PadA7)
- J3 pad A8: Net-(J1-Pad8) -> Net-(J3-PadA8)
- J3 pad A9: Net-(J1-Pad9) -> Net-(J3-PadA9)
- J3 pad B1: Net-(J2-Pad1) -> Net-(J3-PadB1)
- J3 pad B2: Net-(J2-Pad2) -> Net-(J3-PadB2)
- J3 pad B3: Net-(J2-Pad3) -> Net-(J3-PadB3)
- J3 pad B4: Net-(J2-Pad4) -> Net-(J3-PadB4)
- J3 pad B5: Net-(J2-Pad5) -> Net-(J3-PadB5)
- J3 pad B6: Net-(J2-Pad6) -> Net-(J3-PadB6)
- J3 pad B7: Net-(J2-Pad7) -> Net-(J3-PadB7)
- J3 pad B8: Net-(J2-Pad8) -> Net-(J3-PadB8)
- J3 pad B9: Net-(J2-Pad9) -> Net-(J3-PadB9)
Routing:
- net Net-(J3-PadB5): track 0.00 -> 183.7 mm, vias 0 -> 1
- net Net-(J3-PadB9): track 0.00 -> 183.1 mm, vias 0 -> 1
- net Net-(J3-PadB8): track 0.00 -> 175.8 mm, vias 0 -> 1
- net Net-(J3-PadB4): track 0.00 -> 175.5 mm, vias 0 -> 1
- net Net-(J3-PadB7): track 0.00 -> 174.3 mm
- net Net-(J3-PadB3): track 0.00 -> 173.2 mm
- net Net-(J3-PadB6): track 0.00 -> 170.4 mm
- net Net-(J3-PadB2): track 0.00 -> 169.2 mm
- net Net-(J3-PadA1): track 0.00 -> 168.6 mm
- net Net-(J3-PadA6): track 0.00 -> 168.5 mm
- net Net-(J3-PadB1): track 0.00 -> 165.1 mm
- net Net-(J3-PadA2): track 0.00 -> 163.1 mm
- net Net-(J3-PadA7): track 0.00 -> 163.0 mm
- net Net-(J3-PadA3): track 0.00 -> 160.2 mm
- net Net-(J3-PadA8): track 0.00 -> 160.2 mm
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Other:
- board outline added: 32.9 x 251.1 mm
- board text added: "2.4mm PCB"

Commit message: Corrected routing; title block
Parts:
- moved J1 72.8 mm to (57.5, 59.5)
- moved J2 72.8 mm to (57.5, 28.0)
- moved J3 72.8 mm to (48.2, 262.2)
- moved J4 72.8 mm to (49.5, 23.0)
- moved J5 72.8 mm to (49.5, 86.0)
- moved MECH 72.8 mm to (49.5, 136.0)
- moved MECH 72.8 mm to (49.5, 73.0)
Connections:
- J5 pad 1: Net-(J3-PadA1) -> Net-(J3-PadA5)
- J5 pad 11: Net-(J3-PadA8) -> Net-(J3-PadA7)
- J5 pad 12: Net-(J3-PadB7) -> Net-(J3-PadB8)
- J5 pad 13: Net-(J3-PadA4) -> Net-(J3-PadA2)
- J5 pad 14: Net-(J3-PadB2) -> Net-(J3-PadB4)
- J5 pad 15: Net-(J3-PadA9) -> Net-(J3-PadA6)
- J5 pad 16: Net-(J3-PadB6) -> Net-(J3-PadB9)
- J5 pad 17: Net-(J3-PadA5) -> Net-(J3-PadA1)
- J5 pad 18: Net-(J3-PadB1) -> Net-(J3-PadB5)
- J5 pad 2: Net-(J3-PadB5) -> Net-(J3-PadB1)
- J5 pad 3: Net-(J3-PadA6) -> Net-(J3-PadA9)
- J5 pad 4: Net-(J3-PadB9) -> Net-(J3-PadB6)
- J5 pad 5: Net-(J3-PadA2) -> Net-(J3-PadA4)
- J5 pad 6: Net-(J3-PadB4) -> Net-(J3-PadB2)
- J5 pad 7: Net-(J3-PadA7) -> Net-(J3-PadA8)
- J5 pad 8: Net-(J3-PadB8) -> Net-(J3-PadB7)
Routing:
- net Net-(J3-PadA5): track 149.3 -> 171.0 mm
- net Net-(J3-PadB1): track 165.1 -> 185.4 mm
- net Net-(J3-PadA1): track 168.6 -> 148.7 mm, vias 0 -> 1
- net Net-(J3-PadA9): track 154.9 -> 172.7 mm, vias 0 -> 1
- net Net-(J3-PadB5): track 183.7 -> 166.2 mm, vias 1 -> 2
- net Net-(J3-PadB6): track 170.4 -> 187.2 mm, vias 0 -> 1
- net Net-(J3-PadA4): track 155.1 -> 168.3 mm, vias 0 -> 1
- net Net-(J3-PadB2): track 169.2 -> 181.5 mm, vias 0 -> 1
- net Net-(J3-PadB9): track 183.1 -> 171.2 mm, vias 1 -> 2
- net Net-(J3-PadA6): track 168.5 -> 158.6 mm, vias 0 -> 1
- net Net-(J3-PadA8): track 160.2 -> 168.4 mm, vias 0 -> 1
- net Net-(J3-PadB7): track 174.3 -> 181.8 mm, vias 0 -> 1
- net Net-(J3-PadB4): track 175.5 -> 169.1 mm, vias 1 -> 2
- net Net-(J3-PadA2): track 163.1 -> 157.5 mm, vias 0 -> 1
- net Net-(J3-PadA3): track 160.2 -> 163.8 mm, vias 0 -> 1
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